File: bus/1p3/f.kicad_pcb (KiCad board)
At the start: 2 copper layers, 76.2 x 61 mm, 8 parts, among them J1 bus_power_i, J2 bus_i, J3 bus_i, J4 bus_i

Commit message: voltage regulator for each module
Connections:
- net +5V renamed VP
