File: din/main/channel_16/v1/f.sch (KiCad schematic (older format))
At the start: 77 parts, among them J1 fm16_i, J2 wrs_i, J3 wrs_i, J4 bus_i, J5 selector4_i, U1 LTV-357T, U10 LTV-357T, U11 LTV-357T, U12 LTV-357T, U13 LTV-357T, U15 LTV-357T, U16 LTV-357T, U17 LTV-357T, U18 LTV-357T, U2 LTV-357T, U21 74LS245, U22 74LS245, U3 LTV-357T, U4 LTV-357T, U6 LTV-357T, U7 LTV-357T, U8 LTV-357T, U9 LTV-357T

Commit message: voltage regulator for each module
Parts:
- added J6: power_+5V, plc88:power_i, symbol plc88:power_i
- J4: footprint 1my_elements:Bus88_2x14 -> plc88:bus_im
Connections:
- net labels added: VPBUS
Changed lines of the file:
@@
 Text GLabel 10100 2125 0    50   UnSpc ~ 0
 GND
-Text GLabel 10100 2025 0    50   UnSpc ~ 0
-+5V
 Text GLabel 10100 1825 0    50   UnSpc ~ 0
 CLK
@@
 Text GLabel 10100 825  0    50   UnSpc ~ 0
 GND
-Text GLabel 10100 925  0    50   UnSpc ~ 0
-+5V
 Text GLabel 10800 2125 2    50   UnSpc ~ 0
 GND
-Text GLabel 10800 2025 2    50   UnSpc ~ 0
-+5V
 Text GLabel 10800 825  2    50   UnSpc ~ 0
 GND
-Text GLabel 10800 925  2    50   UnSpc ~ 0
-+5V
 Text GLabel 6950 5650 2    50   UnSpc ~ 0
 GND8_15
@@
 F 0 "J4" H 10450 850 50  0000 C CNN
 F 1 "bus_i" H 10450 759 50  0000 C CNN
-F 2 "1my_elements:Bus88_2x14" H 10300 725 50  0001 C CNN
+F 2 "plc88:bus_im" H 10300 725 50  0001 C CNN
 F 3 "" H 10300 725 50  0001 C CNN
 	1    10200 725
@@
 Wire Wire Line
 	6200 1125 6600 1125
+$Comp
+L plc88:power_i J6
+U 1 1 6430747B
+P 9350 700
+F 0 "J6" H 9475 825 50  0000 L CNN
+F 1 "power_+5V" H 9325 750 50  0000 L CNN
+F 2 "plc88:power_i" H 9350 700 50  0001 C CNN
+F 3 "" H 9350 700 50  0001 C CNN
+	1    9350 700
+	1    0    0    -1
+$EndComp
+Text GLabel 9250 1000 0    50   UnSpc ~ 0
+GND
+Text GLabel 9250 900  0    50   UnSpc ~ 0
++5V
+Text GLabel 9250 800  0    50   UnSpc ~ 0
+VPBUS
+Text GLabel 10100 925  0    50   UnSpc ~ 0
+VPBUS
+Text GLabel 10100 2025 0    50   UnSpc ~ 0
+VPBUS
+Text GLabel 10800 2025 2    50   UnSpc ~ 0
+VPBUS
+Text GLabel 10800 925  2    50   UnSpc ~ 0
+VPBUS
 $EndSCHEMATC
